File: hardware/node.brd (EAGLE design)
At the start: 40.8 x 45.9 mm, 106 parts, among them IC1 MAX1555, Q1 P-MOSFET, U1 ATMEGA32U4, U2 MCP1703CB/TOREX-XC6206, Y1 8MHz

Commit message: Hardware modification
Parts:
- added CHG: WIREPAD1,6/0,8, wirepad:1,6/0,8
- LIPO+, LIPO-: value TPPAD1-13 -> WIREPAD1,6/0,8; device testpad:P1-13 -> wirepad:1,6/0,8
- Q1: value P-MOSFET -> NX2301P
- R7, R8: value (none) -> 10k
- moved LIPO+ 0.63 mm to (7.14, 40.9)
- moved LIPO- 0.63 mm to (4.60, 40.9)
- moved TP12 0.50 mm to (15.7, 11.2)
Connections:
- net N$133: now also CHG.1
- net N$192: now also LIPO+.1; no longer LIPO+.TP
- net SL_GND: now also LIPO-.1; no longer LIPO-.TP
Routing:
- net N$133: track 11.3 -> 12.8 mm
- net N$192: track 13.7 -> 14.5 mm
- net _CHG: track 1.58 -> 2.12 mm
Other:
- outline, holes or cut-outs redrawn
- board text added: "LIPO"
- board text added: "oa node v1.5.x"
- board text removed: "oa node v1.5.0"
