File: hardware/node.sch (EAGLE design)
At the start: 106 parts, among them IC1 MAX1555, Q1 P-MOSFET, U1 ATMEGA32U4, U2 MCP1703CB/TOREX-XC6206, Y1 8MHz

Commit message: Hardware modification
Parts:
- added CHG: WIREPAD1,6/0,8, wirepad:WIREPAD1,6/0,8
- LIPO+, LIPO-: value TPPAD1-13 -> WIREPAD1,6/0,8; device testpad:TPPAD1-13 -> wirepad:WIREPAD1,6/0,8
- Q1: value P-MOSFET -> NX2301P
- R7, R8: value (none) -> 10k
Connections:
- net N$133: now also CHG.P
- net N$192: now also LIPO+.P; no longer LIPO+.TP
- net SL_GND: now also LIPO-.P; no longer LIPO-.TP
Changed lines of the file:
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@@
 <setting verticaltext="up"/>
 </settings>
-<grid distance="0.1" unitdist="inch" unit="inch" style="lines" multiple="1" display="yes" altdistance="0.01" altunitdist="inch" altunit="inch"/>
+<grid distance="0.1" unitdist="inch" unit="inch" style="lines" multiple="1" display="no" altdistance="0.01" altunitdist="inch" altunit="inch"/>
 <layers>
 <layer number="1" name="Top" color="4" fill="1" visible="no" active="no"/>
@@
 <part name="GND1" library="SparkFun" deviceset="GND" device=""/>
 <part name="D1" library="SparkFun" deviceset="LED" device="0603" value="Green"/>
-<part name="Q1" library="SparkFun" deviceset="MOSFET-PCHANNEL" device="" value="P-MOSFET"/>
+<part name="Q1" library="SparkFun" deviceset="MOSFET-PCHANNEL" device="" value="NX2301P"/>
 <part name="D2" library="adafruit" deviceset="DIODE" device="SOD-323F"/>
 <part name="RFMXX" library="LowPowerLab" deviceset="RFM12B_MINPADS" device=""/>
@@
 <part name="TP9" library="testpad" deviceset="TP" device="TP08R"/>
 <part name="TP8" library="testpad" deviceset="TP" device="TP08R"/>
-<part name="R7" library="SparkFun" deviceset="RESISTOR" device="0402-RES"/>
-<part name="R8" library="SparkFun" deviceset="RESISTOR" device="0402-RES"/>
+<part name="R7" library="SparkFun" deviceset="RESISTOR" device="0402-RES" value="10k"/>
+<part name="R8" library="SparkFun" deviceset="RESISTOR" device="0402-RES" value="10k"/>
 <part name="GND4" library="SparkFun" deviceset="GND" device=""/>
 <part name="C4" library="SparkFun" deviceset="CAP" device="0402-CAP" value="1uF"/>
@@
 <part name="D5" library="diode" deviceset="DIODE-" device="SOD523" value="RB751S40"/>
 <part name="D6" library="diode" deviceset="DIODE-" device="SOD523" value="RB751S40"/>
-<part name="LIPO+" library="testpad" deviceset="TP" device="PAD1-13"/>
-<part name="LIPO-" library="testpad" deviceset="TP" device="PAD1-13"/>
 <part name="R9" library="SparkFun" deviceset="RESISTOR" device="0402-RES" value="330"/>
 <part name="D7" library="SparkFun" deviceset="LED" device="0603" value="Green"/>
@@
 <part name="U$56" library="openalarm" deviceset="IOPAD" device=""/>
 <part name="U$57" library="openalarm" deviceset="IOPAD" device=""/>
+<part name="CHG" library="wirepad" deviceset="WIREPAD" device="1,6/0,8"/>
+<part name="LIPO+" library="wirepad" deviceset="WIREPAD" device="1,6/0,8"/>
+<part name="LIPO-" library="wirepad" deviceset="WIREPAD" device="1,6/0,8"/>
 </parts>
 <sheets>
@@
 <instance part="R7" gate="G$1" x="58.42" y="60.96" smashed="yes" rot="R90">
 <attribute name="NAME" x="55.88" y="62.0014" size="1.778" layer="95" rot="R180"/>
-<attribute name="VALUE" x="61.722" y="57.15" size="1.778" layer="96" rot="R90"/>
+<attribute name="VALUE" x="64.77" y="61.722" size="1.778" layer="96" rot="R180"/>
 </instance>
 <instance part="R8" gate="G$1" x="58.42" y="45.72" smashed="yes" rot="R90">
 <attribute name="NAME" x="55.88" y="46.7614" size="1.778" layer="95" rot="R180"/>
-<attribute name="VALUE" x="61.722" y="41.91" size="1.778" layer="96" rot="R90"/>
+<attribute name="VALUE" x="64.77" y="46.482" size="1.778" layer="96" rot="R180"/>
 </instance>
 <instance part="GND4" gate="1" x="58.42" y="35.56"/>
@@
 <instance part="D5" gate="G$1" x="195.58" y="24.13" smashed="yes">
 <attribute name="NAME" x="196.85" y="20.8026" size="1.778" layer="95"/>
-<attribute name="VALUE" x="196.85" y="18.0086" size="1.778" layer="96"/>
+<attribute name="VALUE" x="200.66" y="20.5486" size="1.778" layer="96"/>
 </instance>
 <instance part="D6" gate="G$1" x="185.42" y="24.13" smashed="yes">
 <attribute name="NAME" x="182.88" y="29.6926" size="1.778" layer="95"/>
 <attribute name="VALUE" x="177.8" y="26.8986" size="1.778" layer="96"/>
-</instance>
-<instance part="LIPO+" gate="G$1" x="190.5" y="33.02" smashed="yes">
-<attribute name="NAME" x="184.15" y="34.29" size="1.778" layer="95"/>
-<attribute name="TP_SIGNAL_NAME" x="191.77" y="31.75" size="1.778" layer="97"/>
-</instance>
-<instance part="LIPO-" gate="G$1" x="194.31" y="33.02" smashed="yes">
-<attribute name="NAME" x="194.31" y="34.29" size="1.778" layer="95"/>
-<attribute name="TP_SIGNAL_NAME" x="195.58" y="31.75" size="1.778" layer="97"/>
 </instance>
 <instance part="R9" gate="G$1" x="203.2" y="1.27" smashed="yes" rot="R270">
@@
 <instance part="U$56" gate="G$1" x="90.17" y="58.42" rot="R180"/>
 <instance part="U$57" gate="G$1" x="90.17" y="60.96" rot="R180"/>
+<instance part="CHG" gate="G$1" x="208.28" y="19.05" smashed="yes" rot="R180">
+<attribute name="NAME" x="215.773" y="19.7358" size="1.778" layer="95" rot="R180"/>
+<attribute name="VALUE" x="209.423" y="22.352" size="1.778" layer="96" rot="R180" display="off"/>
+</instance>
+<instance part="LIPO+" gate="G$1" x="190.5" y="33.02" smashed="yes" rot="R270">
+<attribute name="NAME" x="185.547" y="34.8742" size="1.778" layer="95"/>
+<attribute name="VALUE" x="187.198" y="34.163" size="1.778" layer="96" rot="R270" display="off"/>
+</instance>
+<instance part="LIPO-" gate="G$1" x="194.31" y="33.02" smashed="yes" rot="R270">
+<attribute name="NAME" x="193.167" y="34.8742" size="1.778" layer="95"/>
+<attribute name="VALUE" x="191.008" y="34.163" size="1.778" layer="96" rot="R270" display="off"/>
+</instance>
 </instances>
 <busses>
@@
 </segment>
 <segment>
-<pinref part="LIPO-" gate="G$1" pin="TP"/>
 <wire x1="194.31" y1="30.48" x2="194.31" y2="27.94" width="0.1524" layer="91"/>
 <wire x1="194.31" y1="27.94" x2="196.85" y2="27.94" width="0.1524" layer="91"/>
 <label x="196.85" y="27.94" size="1.27" layer="95" xref="yes"/>
+<pinref part="LIPO-" gate="G$1" pin="P"/>
 </segment>
 </net>
@@
 <wire x1="190.5" y1="24.13" x2="193.04" y2="24.13" width="0.1524" layer="91"/>
 <junction x="190.5" y="24.13"/>
-<pinref part="LIPO+" gate="G$1" pin="TP"/>
 <wire x1="190.5" y1="24.13" x2="190.5" y2="30.48" width="0.1524" layer="91"/>
+<pinref part="LIPO+" gate="G$1" pin="P"/>
 </segment>
 </net>
@@
 <wire x1="180.34" y1="19.05" x2="203.2" y2="19.05" width="0.1524" layer="91"/>
 <wire x1="203.2" y1="19.05" x2="203.2" y2="16.51" width="0.1524" layer="91"/>
-</segment>
-</net>
+<wire x1="205.74" y1="19.05" x2="203.2" y2="19.05" width="0.1524" layer="91"/>
+<junction x="203.2" y="19.05"/>
+<pinref part="CHG" gate="G$1" pin="P"/>
+</segment>
+</net>

Commit message: Misc
Other:
- note added: "Ajouter des condos de découplage"
- note removed: "C3, C4, C5 : 0603 -> 0402"
Changed lines of the file:
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@@
 <wire x1="71.12" y1="38.1" x2="71.12" y2="-44.45" width="0.1524" layer="98"/>
 <text x="74.93" y="29.21" size="5.08" layer="98">Interface</text>
-<text x="16.51" y="127" size="3.81" layer="98">C3, C4, C5 : 0603 -&gt; 0402</text>
 <text x="16.51" y="-44.45" size="3.81" layer="98">INT:
 D0, D1, D2, D3, D7</text>
@@
 <wire x1="71.12" y1="38.1" x2="71.12" y2="81.28" width="0.1524" layer="98"/>
 <text x="118.11" y="29.21" size="5.08" layer="98">LiPo Shield</text>
+<text x="15.24" y="124.46" size="3.81" layer="98">Ajouter des condos de découplage</text>
 </plain>
 <instances>
